File: PCB/v1/v1.kicad_sch (KiCad schematic)
At the start: 36 parts, among them J1 Screw_Terminal_01x02, Q2 BC548, SW1 Push Button, SW2 Push Button, U1 4060, U10 7400, U2 4060, U3 CD4026BE, U4 CD4026BE, U5 CD4026BE, U6 CD4026BE, U7 CD4026BE, U8 CD4026BE, Y1 32.768kHz

Commit message: Updated PCB Schematics
Parts:
- added R10, R11, R12, R13, R14, R15, R16, R17, R18, R19, R20, R21, R22, R23, R24, R25, R26, R27, R28, R29, R30, R31, R32, R33, R34, R35, R36, R44, R45, R46, R47, R48, R49, R50, R51, R52, R9: 330R, symbol Device:R
- added R37, R38, R39, R40, R41, R42, R43: R, symbol Device:R
- R5: value 330 -> 330R
Connections:
- net +6V: now also R6.1, R51.2, R52.2
- net at U7.1 (CLK): no longer U5.5 (CARRY_OUT)
- net at U7.10 (A): now also R14.2; no longer AFF5.7 (a)
- net at U7.11 (E): now also R12.1; no longer AFF5.1 (e)
- net at U7.12 (B): now also R9.1; no longer AFF5.6 (b)
- net at U7.13 (C): now also R10.1; no longer AFF5.4 (c)
- net at U7.6 (F): now also R13.1; no longer AFF5.9 (f)
- net at U10.5, U7.7 (G): now also R15.2; no longer AFF5.10 (g)
- net at U7.9 (D): now also R11.1; no longer AFF5.2 (d)
- net at AFF4.2 (d): now also R47.2; no longer U6.9 (D)
- net at AFF4.4 (c): now also R46.2; no longer U6.13 (C)
- net at AFF4.5 (DP): now also R52.1
- net at AFF4.6 (b): now also R45.2; no longer U6.12 (B)
- net at AFF4.7 (a): now also R44.2; no longer U6.10 (A)
- net at D1.1 (K), Q2.1 (C): no longer U3.1 (CLK)
- net at AFF5.5 (DP): now also R51.1
- net at U3.10 (A): now also R30.1; no longer AFF2.7 (a)
- net at U3.12 (B): now also R31.1; no longer AFF2.6 (b)
- net at U3.13 (C): now also R32.1; no longer AFF2.4 (c)
- net at U3.9 (D): now also R33.1; no longer AFF2.2 (d)
- net at U6.1 (CLK): no longer U4.5 (CARRY_OUT)
- net at U8.11 (E): now also R20.1; no longer AFF6.1 (e)
- net at AFF6.10 (g): now also R22.2; no longer U8.7 (G)
- net at U8.9 (D): now also R19.1; no longer AFF6.2 (d)
- net at AFF6.4 (c): now also R18.2; no longer U8.13 (C)
- net at U8.12 (B): now also R17.1; no longer AFF6.6 (b)
- net at U10.1, U10.2, U8.10 (A): now also R16.1; no longer AFF6.7 (a)
- net at AFF6.9 (f): now also R21.2; no longer U8.6 (F)
- net at U5.10 (A): now also R37.1; no longer AFF3.7 (a)
- net at U5.11 (E): now also D5.1 (K), R41.1; no longer AFF3.1 (e)
- net at U5.12 (B): now also R38.1; no longer AFF3.6 (b)
- net at U5.13 (C): now also R39.1; no longer AFF3.4 (c)
- net at U5.6 (F): now also D6.1 (K), R42.1; no longer AFF3.9 (f)
- net at U5.7 (G): now also D7.1 (K), R43.1; no longer AFF3.10 (g)
- net at U5.9 (D): now also R40.1; no longer AFF3.2 (d)
- net at U4.10 (A): now also R23.1; no longer AFF1.7 (a)
- net at U4.11 (E): now also D2.1 (K), R27.1; no longer AFF1.1 (e)
- net at U4.12 (B): now also R24.1; no longer AFF1.6 (b)
- net at U4.13 (C): now also R25.1; no longer AFF1.4 (c)
- net at U4.6 (F): now also D3.1 (K), R28.1; no longer AFF1.9 (f)
- net at U4.7 (G): now also D4.1 (K), R29.1; no longer AFF1.10 (g)
- net at U4.9 (D): now also R26.1; no longer AFF1.2 (d)
- new net: AFF3.6 (b), R38.2
- new net: R49.1, U6.6 (F)
- new net: AFF4.9 (f), R49.2
- new net: AFF5.4 (c), R10.2
- new net: AFF4.1 (e), R48.2
- new net: AFF4.10 (g), R50.2
- new net: AFF6.2 (d), R19.2
- new net: AFF5.10 (g), R15.1
- new net: AFF2.7 (a), R30.2
- new net: AFF1.4 (c), R25.2
- new net: AFF5.6 (b), R9.2
- new net: R35.1, U3.6 (F)
- new net: AFF2.9 (f), R35.2
- new net: AFF1.1 (e), R27.2
- new net: AFF1.2 (d), R26.2
- new net: R48.1, U6.11 (E)
- new net: AFF6.6 (b), R17.2
- new net: AFF5.1 (e), R12.2
- new net: AFF5.2 (d), R11.2
- new net: AFF5.7 (a), R14.1
- new net: AFF5.9 (f), R13.2
- new net: R47.1, U6.9 (D)
- new net: AFF2.2 (d), R33.2
- new net: AFF6.7 (a), R16.2
- new net: R34.1, U3.11 (E)
- new net: R36.1, U3.7 (G)
- new net: AFF6.1 (e), R20.2
- new net: R44.1, U6.10 (A)
- new net: R45.1, U6.12 (B)
- new net: R46.1, U6.13 (C)
- new net: R50.1, U6.7 (G)
- new net: AFF2.10 (g), R36.2
- new net: AFF1.6 (b), R24.2
- new net: AFF1.9 (f), R28.2
- new net: AFF2.4 (c), R32.2
- new net: AFF3.4 (c), R39.2
- new net: R22.1, U8.7 (G)
- new net: AFF1.7 (a), R23.2
- new net: AFF3.10 (g), R43.2
- new net: AFF3.9 (f), R42.2
- new net: AFF3.1 (e), R41.2
- new net: AFF3.7 (a), R37.2
- new net: R18.1, U8.13 (C)
- new net: R21.1, U8.6 (F)
- new net: AFF3.2 (d), R40.2
- new net: AFF1.10 (g), R29.2
- new net: AFF2.6 (b), R31.2
- new net: AFF2.1 (e), R34.2
- no-connect marks 0 -> 35
Other:
- note added: "CLK - Mod-12"
- note added: "CLK - Mod-60 (1)"
- note added: "CLK - Mod-60 (2)"
- note added: "Power Supply"
- moved on the sheet: AFF1, AFF2, AFF3, AFF4, AFF5, AFF6, C1, D1, D2, D3, D4, D5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
